File: PCB/HB-RC-4-TOUCH.kicad_pcb (KiCad board)
At the start: 2 copper layers, 261.2 x 53.5 mm, 13 parts, among them J1 Pad1, J2 Pad2, J3 Pad3, J4 Pad4, J5 SCL, J6 SDA, SW1 Config, U1 CC1101, U2 MPR121_Module-Touchpad, X1 Arduino_Pro_Mini

Commit message: update pcb
Parts:
- moved U2 17.5 mm to (227.0, 52.5), turned to 180 degrees
- moved J5 8.96 mm to (228.2, 38.9), turned to 180 degrees
- moved J6 8.96 mm to (225.8, 38.9), turned to 180 degrees
- moved J1 5.90 mm to (46.1, 41.1)
- moved J2 5.90 mm to (93.1, 41.1)
- moved J3 5.90 mm to (140.1, 41.1)
- moved J4 5.90 mm to (187.1, 41.1)
- moved U1 5.20 mm to (258.9, 49.0)
- moved D1 2.65 mm to (277.6, 24.7)
Connections:
- U1 pad 5: Net-(U1-Pad5) -> MISO
- U1 pad 6: MISO -> Net-(U1-Pad6)
Routing:
- net +3V3: track 80.9 -> 54.2 mm
- net GND: track 77.1 -> 99.4 mm
- net Net-(J1-Pad1): track 204.3 -> 188.9 mm
- net Net-(J3-Pad1): track 102.5 -> 88.2 mm
- net Net-(J2-Pad1): track 153.5 -> 139.2 mm
- net Net-(J4-Pad1): track 52.1 -> 43.2 mm
- net MISO: track 26.7 -> 18.2 mm
- net SCK: track 21.7 -> 15.1 mm
- net MOSI: track 28.6 -> 22.8 mm
- net CC1101_GDO0: track 51.4 -> 46.1 mm
- net CC1101_CS: track 32.9 -> 28.8 mm
- net Net-(D1-Pad3): track 13.0 -> 10.3 mm
- net Net-(D1-Pad1): track 9.55 -> 6.90 mm
- net MPR121_IRQ: track 46.3 -> 44.6 mm
- net Net-(SW1-Pad1): track 13.2 -> 12.0 mm
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Other:
- board size 261.2 x 53.5 mm -> 258.4 x 49.8 mm
